Commit message: Complete Laser senser

File: src/model/urdf/mbotModel.urdf (robot description, URDF)
Before this commit: robot mbot, 9 links, 8 joints
Links:
- added link laser_frame, mass 10.0; collision cylinder length=0.060 radius=0.035; visual cylinder length=0.060 radius=0.035
- added link laser_sensor, mass 10.0; collision box size=0.01 0.01 0.01; visual box size=0.01 0.01 0.01
Joints:
- added joint base_link_to_laser_frame: type fixed, parent base_link, child laser_frame, origin xyz=0 0 0.226
- added joint laser_frame_to_laser_sensor: type fixed, parent laser_frame, child laser_sensor, origin xyz=0.0 0.0 0.010
