Commit message: Add laser sensor in model.

File: src/model/urdf/mbotModel.xacro (robot description, xacro)
@@ -1,4 +1,5 @@
 <?xml version="1.0"?>
-<robot name="mbot">
+<robot name="mbot" xmlns:xacro="http://www.ros.org/wiki/xacro">
+  <xacro:include filename="$(find model)/urdf/mbotModel.gazebo" />
   <material name="black">
     <color rgba="0 0 0 1"/>
@@ -13,5 +14,4 @@
     <visual>
       <geometry>
-        <!-- <mesh filename="file:///home/sopper08/TMP/mbot/src/model/meshes/body.stl"/> -->
         <mesh filename="package://model/meshes/dashgoD1_body.stl"/>
       </geometry>

Commit message: sensor ready

File: src/model/urdf/mbotModel.xacro (robot description, xacro)
@@ -1,5 +1,7 @@
 <?xml version="1.0"?>
 <robot name="mbot" xmlns:xacro="http://www.ros.org/wiki/xacro">
+  <!-- Gazebo: Color & Sensor -->
   <xacro:include filename="$(find model)/urdf/mbotModel.gazebo" />
+  <!-- COLOR -->
   <material name="black">
     <color rgba="0 0 0 1"/>
@@ -49,5 +51,5 @@
     </inertial>
   </link>
-    <link name="right_leg">
+  <link name="right_leg">
     <visual>
       <geometry>
@@ -266,3 +268,4 @@
     <origin xyz="0.0 0.0 0.010"/>
   </joint>
+c
 </robot>

Commit message: Control need to be finish

File: src/model/urdf/mbotModel.xacro (robot description, xacro)
@@ -13,4 +13,6 @@
     <color rgba="1.0 1.0 1.0 1.0"/>
   </material>
+  <!-- links -->
+  <link name="dummy"></link>
   <link name="base_link">
     <visual>
@@ -218,13 +220,22 @@
     </inertial>
   </link>
-  <joint name="base_link_to_left_leg" type="continuous">
+  <!-- joints -->
+  <joint name="dummy_joint" type="fixed">
+     <parent link="dummy"/>
+     <child link="base_link"/>
+   </joint>
+  <joint name="left_motor" type="continuous">
     <parent link="base_link"/>
     <child link="left_leg"/>
-    <origin xyz="0 0 0.0625"/>
-  </joint>
-  <joint name="base_link_to_right_leg" type="continuous">
+    <origin xyz="0 0 0.0625" rpy="0 0 0"/>
+    <axis xyz="0 1 0"/>
+    <dynamics damping="0.7"/>
+  </joint>
+  <joint name="right_motor" type="continuous">
     <parent link="base_link"/>
     <child link="right_leg"/>
-    <origin xyz="0 0 0.0625"/>
+    <origin xyz="0 0 0.0625" rpy="0 0 0"/>
+    <axis xyz="0 1 0"/>
+    <dynamics damping="0.7"/>
   </joint>
   <joint name="base_link_to_front_support_of_steering_wheel_frame" type="fixed">
@@ -268,4 +279,24 @@
     <origin xyz="0.0 0.0 0.010"/>
   </joint>
-c
+  <!-- transmissions -->
+  <transmission name="tran1">
+    <type>transmission_interface/SimpleTransmission</type>
+    <joint name="left_motor">
+      <hardwareInterface>hardware_interface/EffortJointInterface</hardwareInterface>
+    </joint>
+    <actuator name="left_leg">
+      <hardwareInterface>hardware_interface/EffortJointInterface</hardwareInterface>
+      <mechanicalReduction>1</mechanicalReduction>
+    </actuator>
+  </transmission>
+  <transmission name="tran2">
+    <type>transmission_interface/SimpleTransmission</type>
+    <joint name="right_motor">
+      <hardwareInterface>hardware_interface/EffortJointInterface</hardwareInterface>
+    </joint>
+    <actuator name="right_leg">
+      <hardwareInterface>hardware_interface/EffortJointInterface</hardwareInterface>
+      <mechanicalReduction>1</mechanicalReduction>
+    </actuator>
+  </transmission>
 </robot>

Commit message: Motor controller finish

File: src/model/urdf/mbotModel.xacro (robot description, xacro)
@@ -229,5 +229,5 @@
     <child link="left_leg"/>
     <origin xyz="0 0 0.0625" rpy="0 0 0"/>
-    <axis xyz="0 1 0"/>
+    <axis xyz="1 0 0"/>
     <dynamics damping="0.7"/>
   </joint>
@@ -236,5 +236,5 @@
     <child link="right_leg"/>
     <origin xyz="0 0 0.0625" rpy="0 0 0"/>
-    <axis xyz="0 1 0"/>
+    <axis xyz="1 0 0"/>
     <dynamics damping="0.7"/>
   </joint>
@@ -283,8 +283,8 @@
     <type>transmission_interface/SimpleTransmission</type>
     <joint name="left_motor">
-      <hardwareInterface>hardware_interface/EffortJointInterface</hardwareInterface>
+      <hardwareInterface>hardware_interface/VelocityJointInterface</hardwareInterface>
     </joint>
     <actuator name="left_leg">
-      <hardwareInterface>hardware_interface/EffortJointInterface</hardwareInterface>
+      <hardwareInterface>hardware_interface/VelocityJointInterface</hardwareInterface>
       <mechanicalReduction>1</mechanicalReduction>
     </actuator>
@@ -293,8 +293,8 @@
     <type>transmission_interface/SimpleTransmission</type>
     <joint name="right_motor">
-      <hardwareInterface>hardware_interface/EffortJointInterface</hardwareInterface>
+      <hardwareInterface>hardware_interface/VelocityJointInterface</hardwareInterface>
     </joint>
     <actuator name="right_leg">
-      <hardwareInterface>hardware_interface/EffortJointInterface</hardwareInterface>
+      <hardwareInterface>hardware_interface/VelocityJointInterface</hardwareInterface>
       <mechanicalReduction>1</mechanicalReduction>
     </actuator>

Commit message: gmapping is ok, but direction is wrong

File: src/model/urdf/mbotModel.xacro (robot description, xacro)
@@ -14,5 +14,5 @@
   </material>
   <!-- links -->
-  <link name="dummy"></link>
+  <!-- <link name="dummy"></link> -->
   <link name="base_link">
     <visual>
@@ -207,5 +207,5 @@
         <box size="0.01 0.01 0.01"/>
       </geometry>
-      <origin xyz="0.0 0.0 0.0"/>
+      <origin xyz="0.0 0.0 0.0" rpy="0.0 0.0 0.0"/>
     </visual>
     <collision>
@@ -213,16 +213,17 @@
         <box size="0.01 0.01 0.01"/>
       </geometry>
-      <origin xyz="0.0 0.0 0.0"/>
-    </collision>
-    <inertial>
-      <mass value="10.0"/>
-      <inertia ixx="1.0" ixy="0.0" ixz="0.0" iyy="1.0" iyz="0.0" izz="1.0"/>
+      <origin xyz="0.0 0.0 0.0" rpy="0.0 0.0 0.0"/>
+    </collision>
+    <inertial>
+      <mass value="1e-5" />
+      <origin xyz="0 0 0" rpy="0 0 0"/>
+      <inertia ixx="1e-6" ixy="0" ixz="0" iyy="1e-6" iyz="0" izz="1e-6" />>
     </inertial>
   </link>
   <!-- joints -->
-  <joint name="dummy_joint" type="fixed">
+  <!-- <joint name="dummy_joint" type="fixed">
      <parent link="dummy"/>
      <child link="base_link"/>
-   </joint>
+  </joint> -->
   <joint name="left_motor" type="continuous">
     <parent link="base_link"/>

Commit message: Resolve the problem of orientation of odom

File: src/model/urdf/mbotModel.xacro (robot description, xacro)
@@ -16,4 +16,6 @@
   <!-- <link name="dummy"></link> -->
   <link name="base_link">
+  </link>
+  <link name="body_link">
     <visual>
       <geometry>
@@ -222,10 +224,11 @@
   </link>
   <!-- joints -->
-  <!-- <joint name="dummy_joint" type="fixed">
-     <parent link="dummy"/>
-     <child link="base_link"/>
-  </joint> -->
+  <joint name="base_to_body" type="fixed">
+     <parent link="base_link"/>
+     <child link="body_link"/>
+     <origin xyz="0 0 0" rpy="0 0 1.57075"/>
+  </joint>
   <joint name="left_motor" type="continuous">
-    <parent link="base_link"/>
+    <parent link="body_link"/>
     <child link="left_leg"/>
     <origin xyz="0 0 0.0625" rpy="0 0 0"/>
@@ -234,5 +237,5 @@
   </joint>
   <joint name="right_motor" type="continuous">
-    <parent link="base_link"/>
+    <parent link="body_link"/>
     <child link="right_leg"/>
     <origin xyz="0 0 0.0625" rpy="0 0 0"/>
@@ -240,11 +243,11 @@
     <dynamics damping="0.7"/>
   </joint>
-  <joint name="base_link_to_front_support_of_steering_wheel_frame" type="fixed">
-    <parent link="base_link"/>
+  <joint name="body_link_to_front_support_of_steering_wheel_frame" type="fixed">
+    <parent link="body_link"/>
     <child link="front_support_of_steering_wheel_frame"/>
     <origin xyz="0 -0.130 0.038"/>
   </joint>
-  <joint name="base_link_to_back_support_of_steering_wheel_frame" type="fixed">
-    <parent link="base_link"/>
+  <joint name="body_link_to_back_support_of_steering_wheel_frame" type="fixed">
+    <parent link="body_link"/>
     <child link="back_support_of_steering_wheel_frame"/>
     <origin xyz="0 0.130 0.038"/>
@@ -270,6 +273,6 @@
     <origin xyz="0.0 -0.005 -0.0255"/>
   </joint>
-  <joint name="base_link_to_laser_frame" type="fixed">
-    <parent link="base_link"/>
+  <joint name="body_link_to_laser_frame" type="fixed">
+    <parent link="body_link"/>
     <child link="laser_frame"/>
     <origin xyz="0 0 0.226"/>
@@ -278,5 +281,5 @@
     <parent link="laser_frame"/>
     <child link="laser_sensor"/>
-    <origin xyz="0.0 0.0 0.010"/>
+    <origin xyz="0.0 0.0 0.010" rpy="0.0 0.0 0.0" />
   </joint>
   <!-- transmissions -->

Commit message: Fuckin parameters

File: src/model/urdf/mbotModel.xacro (robot description, xacro)
@@ -14,7 +14,8 @@
   </material>
   <!-- links -->
-  <!-- <link name="dummy"></link> -->
   <link name="base_link">
   </link>
+  <link name="base_footprint">
+  </link>
   <link name="body_link">
     <visual>
@@ -22,5 +23,5 @@
         <mesh filename="package://model/meshes/dashgoD1_body.stl"/>
       </geometry>
-      <origin rpy="0 3.1415 1.57075" xyz="0.203 0.203 0.196 "/>
+      <origin rpy="0 3.14159265359 1.57079632679" xyz="0.203 0.203 0.196 "/>
       <material name="black"/>
     </visual>
@@ -29,5 +30,5 @@
         <mesh filename="package://model/meshes/dashgoD1_body.stl"/>
       </geometry>
-      <origin rpy="0 3.1415 1.57075" xyz="0.203 0.203 0.196 "/>
+      <origin rpy="0 3.14159265359 1.57079632679" xyz="0.203 0.203 0.196 "/>
     </collision>
     <inertial>
@@ -41,5 +42,5 @@
         <cylinder length="0.035" radius="0.0625"/>
       </geometry>
-      <origin rpy="0 1.57075 0" xyz="0.17535 0 0"/>
+      <origin rpy="0 1.57079632679 0" xyz="0 0 0"/>
       <material name="gray"/>
     </visual>
@@ -48,5 +49,5 @@
         <cylinder length="0.035" radius="0.0625"/>
       </geometry>
-      <origin rpy="0 1.57075 0" xyz="0.17535 0 0"/>
+      <origin rpy="0 1.57079632679 0" xyz="0 0 0"/>
     </collision>
     <inertial>
@@ -60,5 +61,5 @@
         <cylinder length="0.035" radius="0.0625"/>
       </geometry>
-      <origin rpy="0 1.57075 0" xyz="-0.17535 0 0"/>
+      <origin rpy="0 1.57079632679 0" xyz="-0 0 0"/>
       <material name="gray"/>
     </visual>
@@ -67,5 +68,5 @@
         <cylinder length="0.035" radius="0.0625"/>
       </geometry>
-      <origin rpy="0 1.57075 0" xyz="-0.17535 0 0"/>
+      <origin rpy="0 1.57079632679 0" xyz="-0 0 0"/>
     </collision>
     <inertial>
@@ -117,5 +118,5 @@
         <mesh filename="package://model/meshes/dashgoD1_steering_wheel_frame.stl"/>
       </geometry>
-      <origin rpy="1.57075 0 1.57075" xyz="-0.0095 -0.017 -0.0375"/>
+      <origin rpy="1.57079632679 0 1.57079632679" xyz="-0.0095 -0.017 -0.0375"/>
     </visual>
     <collision>
@@ -123,5 +124,5 @@
         <mesh filename="package://model/meshes/dashgoD1_steering_wheel_frame.stl"/>
       </geometry>
-      <origin rpy="1.57075 0 1.57075" xyz="-0.0095 -0.017 -0.0375"/>
+      <origin rpy="1.57079632679 0 1.57079632679" xyz="-0.0095 -0.017 -0.0375"/>
     </collision>
     <inertial>
@@ -135,5 +136,5 @@
         <mesh filename="package://model/meshes/dashgoD1_steering_wheel_frame.stl"/>
       </geometry>
-      <origin rpy="1.57075 0 1.57075" xyz="-0.0095 -0.017 -0.0375"/>
+      <origin rpy="1.57079632679 0 1.57079632679" xyz="-0.0095 -0.017 -0.0375"/>
     </visual>
     <collision>
@@ -141,5 +142,5 @@
         <mesh filename="package://model/meshes/dashgoD1_steering_wheel_frame.stl"/>
       </geometry>
-      <origin rpy="1.57075 0 1.57075" xyz="-0.0095 -0.017 -0.0375"/>
+      <origin rpy="1.57079632679 0 1.57079632679" xyz="-0.0095 -0.017 -0.0375"/>
     </collision>
     <inertial>
@@ -153,5 +154,5 @@
         <cylinder radius="0.0125" length="0.015"/>
       </geometry>
-      <origin rpy="0 1.57075 0" xyz="0 0 0"/>
+      <origin rpy="0 1.57079632679 0" xyz="0 0 0"/>
       <material name="white"/>
     </visual>
@@ -160,5 +161,5 @@
         <cylinder radius="0.0125" length="0.015"/>
       </geometry>
-      <origin rpy="0 1.57075 0" xyz="0 0 0"/>
+      <origin rpy="0 1.57079632679 0" xyz="0 0 0"/>
     </collision>
     <inertial>
@@ -172,5 +173,5 @@
         <cylinder radius="0.0125" length="0.015"/>
       </geometry>
-      <origin rpy="0 1.57075 0" xyz="0 0 0"/>
+      <origin rpy="0 1.57079632679 0" xyz="0 0 0"/>
       <material name="white"/>
     </visual>
@@ -179,5 +180,5 @@
         <cylinder radius="0.0125" length="0.015"/>
       </geometry>
-      <origin rpy="0 1.57075 0" xyz="0 0 0"/>
+      <origin rpy="0 1.57079632679 0" xyz="0 0 0"/>
     </collision>
     <inertial>
@@ -227,10 +228,15 @@
      <parent link="base_link"/>
      <child link="body_link"/>
-     <origin xyz="0 0 0" rpy="0 0 1.57075"/>
+     <origin xyz="0 0 0" rpy="0 0 1.57079632679"/>
+  </joint>
+  <joint name="footprint_to_base" type="fixed">
+     <parent link="base_footprint"/>
+     <child link="base_link"/>
+     <origin xyz="0 0 0" rpy="0 0 0"/>
   </joint>
   <joint name="left_motor" type="continuous">
     <parent link="body_link"/>
     <child link="left_leg"/>
-    <origin xyz="0 0 0.0625" rpy="0 0 0"/>
+    <origin xyz="0.17535 0 0.0625" rpy="0 0 0"/>
     <axis xyz="1 0 0"/>
     <dynamics damping="0.7"/>
@@ -239,5 +245,5 @@
     <parent link="body_link"/>
     <child link="right_leg"/>
-    <origin xyz="0 0 0.0625" rpy="0 0 0"/>
+    <origin xyz="-0.17535 0 0.0625" rpy="0 0 0"/>
     <axis xyz="1 0 0"/>
     <dynamics damping="0.7"/>

Commit message: Fucking steering wheel

File: src/model/urdf/mbotModel.xacro (robot description, xacro)
@@ -33,5 +33,5 @@
     </collision>
     <inertial>
-      <mass value="10.0"/>
+      <mass value="50.0"/>
       <inertia ixx="1.0" ixy="0.0" ixz="0.0" iyy="1.0" iyz="0.0" izz="1.0"/>
     </inertial>
@@ -90,5 +90,5 @@
     </collision>
     <inertial>
-      <mass value="10.0"/>
+      <mass value="1.0"/>
       <inertia ixx="1.0" ixy="0.0" ixz="0.0" iyy="1.0" iyz="0.0" izz="1.0"/>
     </inertial>
@@ -109,5 +109,5 @@
     </collision>
     <inertial>
-      <mass value="10.0"/>
+      <mass value="1.0"/>
       <inertia ixx="1.0" ixy="0.0" ixz="0.0" iyy="1.0" iyz="0.0" izz="1.0"/>
     </inertial>
@@ -127,5 +127,5 @@
     </collision>
     <inertial>
-      <mass value="10.0"/>
+      <mass value="1.0"/>
       <inertia ixx="1.0" ixy="0.0" ixz="0.0" iyy="1.0" iyz="0.0" izz="1.0"/>
     </inertial>
@@ -145,9 +145,9 @@
     </collision>
     <inertial>
-      <mass value="10.0"/>
-      <inertia ixx="1.0" ixy="0.0" ixz="0.0" iyy="1.0" iyz="0.0" izz="1.0"/>
-    </inertial>
-  </link>
-  <link name="front_steering_wheel">
+      <mass value="1.0"/>
+      <inertia ixx="1.0" ixy="0.0" ixz="0.0" iyy="1.0" iyz="0.0" izz="1.0"/>
+    </inertial>
+  </link>
+  <!-- <link name="front_steering_wheel">
     <visual>
       <geometry>
@@ -164,5 +164,5 @@
     </collision>
     <inertial>
-      <mass value="10.0"/>
+      <mass value="1.0"/>
       <inertia ixx="1.0" ixy="0.0" ixz="0.0" iyy="1.0" iyz="0.0" izz="1.0"/>
     </inertial>
@@ -183,8 +183,8 @@
     </collision>
     <inertial>
-      <mass value="10.0"/>
-      <inertia ixx="1.0" ixy="0.0" ixz="0.0" iyy="1.0" iyz="0.0" izz="1.0"/>
-    </inertial>
-  </link>
+      <mass value="1.0"/>
+      <inertia ixx="1.0" ixy="0.0" ixz="0.0" iyy="1.0" iyz="0.0" izz="1.0"/>
+    </inertial>
+  </link> -->
   <link name="laser_frame">
     <visual>
@@ -201,5 +201,5 @@
     </collision>
     <inertial>
-      <mass value="10.0"/>
+      <mass value="1.0"/>
       <inertia ixx="1.0" ixy="0.0" ixz="0.0" iyy="1.0" iyz="0.0" izz="1.0"/>
     </inertial>
@@ -269,14 +269,14 @@
     <origin xyz="0 0 0"/>
   </joint>
-  <joint name="front_steering_wheel_frame_to_wheel" type="continuous">
+  <!-- <joint name="front_steering_wheel_frame_to_wheel" type="floating">
     <parent link="front_steering_wheel_frame"/>
     <child link="front_steering_wheel"/>
     <origin xyz="0.0 -0.005 -0.0255"/>
   </joint>
-  <joint name="back_steering_wheel_frame_to_wheel" type="continuous">
+  <joint name="back_steering_wheel_frame_to_wheel" type="floating">
     <parent link="back_steering_wheel_frame"/>
     <child link="back_steering_wheel"/>
     <origin xyz="0.0 -0.005 -0.0255"/>
-  </joint>
+  </joint> -->
   <joint name="body_link_to_laser_frame" type="fixed">
     <parent link="body_link"/>

Commit message: Not bad parameters

File: src/model/urdf/mbotModel.xacro (robot description, xacro)
@@ -28,11 +28,13 @@
     <collision>
       <geometry>
-        <mesh filename="package://model/meshes/dashgoD1_body.stl"/>
-      </geometry>
-      <origin rpy="0 3.14159265359 1.57079632679" xyz="0.203 0.203 0.196 "/>
-    </collision>
-    <inertial>
-      <mass value="50.0"/>
-      <inertia ixx="1.0" ixy="0.0" ixz="0.0" iyy="1.0" iyz="0.0" izz="1.0"/>
+        <!-- <mesh filename="package://model/meshes/dashgoD1_body.stl"/> -->
+        <cylinder length="0.158" radius="0.203"/>
+      </geometry>
+      <!-- <origin rpy="0 3.14159265359 1.57079632679" xyz="0.203 0.203 0.196 "/> -->
+      <origin rpy="0 0 0" xyz="0 0 0.117 "/>
+    </collision>
+    <inertial>
+      <mass value="15.0"/>
+      <inertia ixx="0.352" ixy="0.0" ixz="0.0" iyy="0.352" iyz="0.0" izz="0.309"/>
     </inertial>
   </link>
@@ -53,5 +55,5 @@
     <inertial>
       <mass value="10.0"/>
-      <inertia ixx="1.0" ixy="0.0" ixz="0.0" iyy="1.0" iyz="0.0" izz="1.0"/>
+      <inertia ixx="0.01" ixy="0.0" ixz="0.0" iyy="0.01" iyz="0.0" izz="0.01"/>
     </inertial>
   </link>
@@ -72,5 +74,5 @@
     <inertial>
       <mass value="10.0"/>
-      <inertia ixx="1.0" ixy="0.0" ixz="0.0" iyy="1.0" iyz="0.0" izz="1.0"/>
+      <inertia ixx="0.01" ixy="0.0" ixz="0.0" iyy="0.01" iyz="0.0" izz="0.01"/>
     </inertial>
   </link>
@@ -91,5 +93,5 @@
     <inertial>
       <mass value="1.0"/>
-      <inertia ixx="1.0" ixy="0.0" ixz="0.0" iyy="1.0" iyz="0.0" izz="1.0"/>
+      <inertia ixx="0.01" ixy="0.0" ixz="0.0" iyy="0.01" iyz="0.0" izz="0.01"/>
     </inertial>
   </link>
@@ -110,5 +112,5 @@
     <inertial>
       <mass value="1.0"/>
-      <inertia ixx="1.0" ixy="0.0" ixz="0.0" iyy="1.0" iyz="0.0" izz="1.0"/>
+      <inertia ixx="0.01" ixy="0.0" ixz="0.0" iyy="0.01" iyz="0.0" izz="0.01"/>
     </inertial>
   </link>
@@ -128,5 +130,5 @@
     <inertial>
       <mass value="1.0"/>
-      <inertia ixx="1.0" ixy="0.0" ixz="0.0" iyy="1.0" iyz="0.0" izz="1.0"/>
+      <inertia ixx="0.01" ixy="0.0" ixz="0.0" iyy="0.01" iyz="0.0" izz="0.01"/>
     </inertial>
   </link>
@@ -146,8 +148,8 @@
     <inertial>
       <mass value="1.0"/>
-      <inertia ixx="1.0" ixy="0.0" ixz="0.0" iyy="1.0" iyz="0.0" izz="1.0"/>
-    </inertial>
-  </link>
-  <!-- <link name="front_steering_wheel">
+      <inertia ixx="0.01" ixy="0.0" ixz="0.0" iyy="0.01" iyz="0.0" izz="0.01"/>
+    </inertial>
+  </link>
+  <link name="front_steering_wheel">
     <visual>
       <geometry>
@@ -165,5 +167,5 @@
     <inertial>
       <mass value="1.0"/>
-      <inertia ixx="1.0" ixy="0.0" ixz="0.0" iyy="1.0" iyz="0.0" izz="1.0"/>
+      <inertia ixx="0.01" ixy="0.0" ixz="0.0" iyy="0.01" iyz="0.0" izz="0.01"/>
     </inertial>
   </link>
@@ -184,7 +186,7 @@
     <inertial>
       <mass value="1.0"/>
-      <inertia ixx="1.0" ixy="0.0" ixz="0.0" iyy="1.0" iyz="0.0" izz="1.0"/>
-    </inertial>
-  </link> -->
+      <inertia ixx="0.01" ixy="0.0" ixz="0.0" iyy="0.01" iyz="0.0" izz="0.01"/>
+    </inertial>
+  </link>
   <link name="laser_frame">
     <visual>
@@ -202,5 +204,5 @@
     <inertial>
       <mass value="1.0"/>
-      <inertia ixx="1.0" ixy="0.0" ixz="0.0" iyy="1.0" iyz="0.0" izz="1.0"/>
+      <inertia ixx="0.01" ixy="0.0" ixz="0.0" iyy="0.01" iyz="0.0" izz="0.01"/>
     </inertial>
   </link>
@@ -269,14 +271,14 @@
     <origin xyz="0 0 0"/>
   </joint>
-  <!-- <joint name="front_steering_wheel_frame_to_wheel" type="floating">
+  <joint name="front_steering_wheel_frame_to_wheel" type="fixed">
     <parent link="front_steering_wheel_frame"/>
     <child link="front_steering_wheel"/>
     <origin xyz="0.0 -0.005 -0.0255"/>
   </joint>
-  <joint name="back_steering_wheel_frame_to_wheel" type="floating">
+  <joint name="back_steering_wheel_frame_to_wheel" type="fixed">
     <parent link="back_steering_wheel_frame"/>
     <child link="back_steering_wheel"/>
     <origin xyz="0.0 -0.005 -0.0255"/>
-  </joint> -->
+  </joint>
   <joint name="body_link_to_laser_frame" type="fixed">
     <parent link="body_link"/>
